Commit message: update

File: src/amr/description/amr_description.urdf (robot description, URDF)
Before this commit: robot amr, 7 links, 6 joints
Links:
- link chassis: geometry visual box size=0.5 0.42 0.52
- link wheel_left_link: geometry collision cylinder length=0.046 radius=0; visual cylinder length=0.046 radius=0.065
- link wheel_right_link: geometry collision cylinder length=0.046 radius=0.065; visual cylinder length=0.046 radius=0.065
Joints:
- joint lidar1_joint: origin xyz=0.345 0.0 0.04 rpy=3.14 0 -3.14 -> xyz=0.26 0.0 0.225 rpy=3.14 0 -3.14
- joint lidar2_joint: origin xyz=-0.345 -0.0 0.04 rpy=3.14 0 0 -> xyz=-0.26 -0.0 0.225 rpy=3.14 0 0
- joint lidar_joint: origin xyz=0.0 0.0 0.04 rpy=3.14 0 -3.14 -> xyz=0.0 0.0 0.225 rpy=3.14 0 -3.14
- joint wheel_left_joint: origin xyz=0 0.145 0.085 rpy=-1.57 0 0 -> xyz=0 0.1 0.065 rpy=-1.57 0 0
- joint wheel_right_joint: origin xyz=0 -0.145 0.085 rpy=1.57 0 0 -> xyz=0 -0.1 0.065 rpy=1.57 0 0
